Commit message: added parent link, origin to urdf, parameterized launch file

File: robotiq_description/urdf/robotiq_2f_140_gripper.urdf.xacro (robot description, xacro)
@@ -4,9 +4,15 @@
     <xacro:arg name="use_fake_hardware" default="true" />
     <xacro:arg name="com_port" default="/dev/ttyUSB0" />
+    <xacro:arg name="parent" default="world" />
+    <xacro:arg name="origin" default="0 0 0 0 0 0" />
+    <!-- Split the origin into xyz and rpy -->
+    <xacro:property name="origin_clean" value="${'$(arg origin)'.replace('&quot;', '')}" />
+    <xacro:property name="origin_xyz" value="${origin_clean.split()[0:3]}" />
+    <xacro:property name="origin_rpy" value="${origin_clean.split()[3:6]}" />
     <!-- Import macros -->
     <xacro:include filename="$(find robotiq_description)/urdf/robotiq_2f_140_macro.urdf.xacro" />
-    <link name="world" />
-    <xacro:robotiq_gripper name="RobotiqGripperHardwareInterface" prefix="" parent="world" use_fake_hardware="$(arg use_fake_hardware)" com_port="$(arg com_port)">
-        <origin xyz="0 0 0" rpy="0 0 0" />
+    <link name="$(arg parent)" />
+    <xacro:robotiq_gripper name="RobotiqGripperHardwareInterface" prefix="" parent="$(arg parent)" use_fake_hardware="$(arg use_fake_hardware)" com_port="$(arg com_port)">
+        <origin xyz="${' '.join(origin_xyz)}" rpy="${' '.join(origin_rpy)}" />
     </xacro:robotiq_gripper>
 </robot>

File: robotiq_description/urdf/robotiq_2f_85_gripper.urdf.xacro (robot description, xacro)
@@ -4,9 +4,15 @@
     <xacro:arg name="use_fake_hardware" default="true" />
     <xacro:arg name="com_port" default="/dev/ttyUSB0" />
+    <xacro:arg name="parent" default="world" />
+    <xacro:arg name="origin" default="0 0 0 0 0 0" />
+    <!-- Split the origin into xyz and rpy -->
+    <xacro:property name="origin_clean" value="${'$(arg origin)'.replace('&quot;', '')}" />
+    <xacro:property name="origin_xyz" value="${origin_clean.split()[0:3]}" />
+    <xacro:property name="origin_rpy" value="${origin_clean.split()[3:6]}" />
     <!-- Import macros -->
     <xacro:include filename="$(find robotiq_description)/urdf/robotiq_2f_85_macro.urdf.xacro" />
-    <link name="world" />
-    <xacro:robotiq_gripper name="RobotiqGripperHardwareInterface" prefix="" parent="world" use_fake_hardware="$(arg use_fake_hardware)" com_port="$(arg com_port)">
-        <origin xyz="0 0 0" rpy="0 0 0" />
+    <link name="$(arg parent)" />
+    <xacro:robotiq_gripper name="RobotiqGripperHardwareInterface" prefix="" parent="$(arg parent)" use_fake_hardware="$(arg use_fake_hardware)" com_port="$(arg com_port)">
+        <origin xyz="${' '.join(origin_xyz)}" rpy="${' '.join(origin_rpy)}" />
     </xacro:robotiq_gripper>
 </robot>
